File: hardware/rpi-camera-led.kicad_sch (KiCad schematic)
At the start: 20 parts, among them J1 FFC 15P 1.0mm bottom contact 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, J2 FFC 15P 1.0mm top contact (to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, J3 Qwiic (JST SH 1.0mm), J4 SWD program header 2.54mm, Q1 AO3400A, Q2 Phototransistor, U1 CH32V003A4M6

Commit message: Actually reverse J2's pin order, which a708eef only implied
a708eef swapped J2 to the top-contact part and claimed that made the
bus route straight.  It did not.  The two variants share one land
pattern, so changing the part moved no pad and altered no net: the
board was byte-identical in every way that matters and every
pass-through net still had to cross the bus.  Tim spotted it -- the
connector did not seem to have changed because nothing had.

The reversal has to live in the net mapping, and now does.  Measured
from the board rather than assumed: J1 sits at -90 degrees and J2 at
+90, so J1 pad k is physically opposite J2 pad 16-k (J1.1 faces J2.15,
J1.8 faces J2.8, dy 0.049mm).  A net can only be a straight trace if it
joins such a pair.

Dropping (mirror x) from J2's symbol does exactly that and nothing
else: the pin numbering reverses against labels and wires that all stay
where they are, so J2.m now carries what J1.(16-m) does.  That is also
what the top-contact part buys -- its cable goes in flipped, so contact
m really does land on the conductor the Pi calls 16-m.  The two changes
are one change; a708eef was half of it.

On the sheet the two connectors' pin numbers now run in opposite
directions, which is the honest picture: every net's label lines up
horizontally across the gap.

check_schematic.py gains that as a standing invariant rather than a
one-off measurement -- it now fails any net where J1.k does not face
J2.(16-k), the GPIO channels pairing through R6/R7 by name.  Checked
against the pre-fix schematic, where it flags 14 of the 15 nets (pin 8
is self-symmetric), so it is not vacuous.

The board's J2 pads follow, 14 reassigned, pad 8 unchanged for the same
reason.  No pad moved; kicad-cli reports schematic_parity 0.  DRC goes
90 -> 92 violations, the delta being two more starved_thermal: GND now
lands on J2 pads 6/9/12/15 instead of 1/4/7/10, so the zone's thermal
spokes fall differently.  Clearance and mask-bridge counts are
unchanged, and all of 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
Connections:
- net 3V3: now also J2.1 (Pin_1); no longer J2.15 (Pin_15)
- net CAM_CK_P: now also J2.7 (Pin_7); no longer J2.9 (Pin_9)
- net CAM_D0_N: now also J2.14 (Pin_14); no longer J2.2 (Pin_2)
- net CAM_D0_P: now also J2.13 (Pin_13); no longer J2.3 (Pin_3)
- net CAM_D1_N: now also J2.11 (Pin_11); no longer J2.5 (Pin_5)
- net CAM_D1_P: now also J2.10 (Pin_10); no longer J2.6 (Pin_6)
- net CAM_IO0: now also J2.5 (Pin_5); no longer J2.11 (Pin_11)
- net CAM_IO1: now also J2.4 (Pin_4); no longer J2.12 (Pin_12)
- net GND: now also J2.12 (Pin_12), J2.15 (Pin_15), J2.6 (Pin_6), J2.9 (Pin_9); no longer J2.1 (Pin_1), J2.10 (Pin_10), J2.4 (Pin_4), J2.7 (Pin_7)
- net SCL: now also J2.3 (Pin_3); no longer J2.13 (Pin_13)
- net SDA: now also J2.2 (Pin_2); no longer J2.14 (Pin_14)
Changed lines of the file:
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@@
 		(lib_id "Connector_Generic:Conn_01x15")
 		(at 74.93 82.55 0)
-		(mirror x)
 		(unit 1)
 		(exclude_from_sim no)
