File: hardware/rpi-camera-led.kicad_pcb (KiCad board)
At the start: 2 copper layers, 25 x 23.9 mm, 20 parts, among them J1 FFC 15P 1.0mm bottom contact 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, J2 FFC 15P 1.0mm top contact (to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, J3 Qwiic (JST SH 1.0mm), J4 SWD program header 2.54mm, Q1 AO3400A, Q2 Phototransistor, U1 CH32V003A4M6

Commit message: Build 3D models for the FFC connectors, and wire both up
KiCad's stock footprint points at
Connector_FFC-FPC.3dshapes/JUSHUO_AFA07-S15FCA-00_...step, which does not
exist.  Not in the snap, and not upstream either: kicad-packages3D ships
112 files in that library and none of them are JUSHUO.  Component Search
Engine has one, but SamacSys's terms do not permit redistribution, so it
cannot go in an Apache-2.0 repository.

So gen_connector_model.py builds one from the manufacturer's drawing,
which we can carry.  Everything dimensioned comes from that drawing or
from KiCad's stock footprint, whose F.Fab outline is the body outline and
whose land pattern was already verified against the drawing pad for pad:
the plan outline from F.Fab, 2.50mm height from the side view and the
"H2.5" in the product name, contact tails on the land pattern itself, and
the colours from note 1 ("Housing: ... Color: natural", "Latch: ...
Color: black").  The envelope comes out 22.00 x 6.95 x 2.50 mm, which is
DIM D, the F.Fab depth and that 2.50 respectively.  The cable slot is the
one invented feature -- the drawing does not dimension it -- and it cuts
only into the front face, so the outside envelope stays exact.

Both STEP and WRL are written.  The WRL scale is not obvious and is easy
to get wrong, so it was measured rather than assumed: a known-good
library model has a WRL Z span of 0.7864 against a STEP Z span of exactly
2.0000, which is the 2.54 factor, and WRL Y is the negation of footprint
Y.

J1 was still on the stock footprint, so it now gets a project copy too --
otherwise half the board would keep referencing a model that isn't there.
Both connectors are now project-local, footprint and model.

What the models immediately show is that both connectors are turned the
wrong way round.  Their housings are flush with the board edges (J1 ends
at x=20.000, J2 at x=45.000, outline 20.0-45.0), which points both mouths
inward, 14.4mm apart, facing each other across the middle of the board.
T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
Parts:
- J1: footprint Connector_FFC-FPC:JUSHUO_AFA07-S15FCA-00_1x15-1MP_P1.0mm_Horizontal -> rpi-camera-led:JUSHUO_AFA07-S15FCA-00_1x15-1MP_P1.0mm_Horizontal
Changed lines of the file:
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@@
 		)
 	)
-	(footprint "Connector_FFC-FPC:JUSHUO_AFA07-S15FCA-00_1x15-1MP_P1.0mm_Horizontal"
+	(footprint "rpi-camera-led:JUSHUO_AFA07-S15FCA-00_1x15-1MP_P1.0mm_Horizontal"
 		(layer "F.Cu")
 		(at 22.825 31.931 -90)
@@
 		)
 		(embedded_fonts no)
-		(model "${KICAD9_3DMODEL_DIR}/Connector_FFC-FPC.3dshapes/JUSHUO_AFA07-S15FCA-00_1x15-1MP_P1.0mm_Horizontal.step"
+		(model "${KIPRJMOD}/rpi-camera-led.3dshapes/JUSHUO_AFA07-S15FCA-00_1x15-1MP_P1.0mm_Horizontal.step"
 			(offset
 				(xyz 0 0 0)
@@
 		)
 		(embedded_fonts no)
-		(model "${KICAD9_3DMODEL_DIR}/Connector_FFC-FPC.3dshapes/JUSHUO_AFA07-S15FCA-00_1x15-1MP_P1.0mm_Horizontal.step"
+		(model "${KIPRJMOD}/rpi-camera-led.3dshapes/JUSHUO_AFA07-S15ECA-00_1x15-1MP_P1.0mm_Horizontal.step"
 			(offset
 				(xyz 0 0 0)
