File: hardware/rpi-camera-led.kicad_pcb (KiCad board)
At the start: 2 copper layers, 25 x 23.9 mm, 20 parts, among them J1 FFC 15P 1.0mm bottom contact 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, J2 FFC 15P 1.0mm top contact (to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, J3 Qwiic (JST SH 1.0mm), J4 SWD program header 2.54mm, Q1 AO3400A, Q2 Phototransistor, U1 CH32V003A4M6

Commit message: Add back the Raspberry Pi camera board's mounting holes
The board uses the Camera Module 2 outline, so it should take the same
screws.  d0c15fe put the holes in; they were lost somewhere after that
and nobody noticed, which is exactly the failure check_pcb.py exists to
catch, so it now verifies the pattern too -- confirmed non-vacuous by
running it against the previous commit's board, where it reports 0 holes
and fails.

Positions are from the official mechanical drawing RP-008149-DS
(RPI-CAM-V2_1): "4x 2.2mm diameter holes", 2mm in from each end of the
25mm axis for a 21.0mm pitch, and 2.0 and 14.5mm from one end of the
23.862mm axis for a 12.5mm pitch.  That second pair is asymmetric on the
camera because its FFC connector eats the far edge; here it is centred,
which is what this board carried before.

Unlike the previous version these use the stock MountingHole_2.2mm_M2
footprint, courtyard and all.  The old code hand-built the holes without
a courtyard, with a comment explaining that the stock one "would collide
with the FFC connector courtyards" -- which is not a footprint problem to
be worked around but a real mechanical conflict that was being silenced.

With a real courtyard DRC says so: four courtyards_overlap errors, one
per hole, taking the count from 17 to 21.  All four holes sit under a
connector housing.  The camera runs its 21.0mm pitch between two bare
edges and puts its one connector on a third; this board has a connector
on both ends of that axis, each 5.30mm deep, so holes 2mm in from each
end land underneath them.  Neither the pattern nor the connectors are
wrong on their own -- they just cannot both fit across 25mm, and the way
out costs something: a longer board, connectors on the 25mm edges, or
holes that no longer match the camera.  Recorded in the README rather
than resolved, because that is a design decision.

Co-Authored-By: Claude Opus 5 <noreply@anthropic.com>
Claude-Session: https://claude.ai/code/session_01NAtQfzwuXNuQMrD3BxPvxL
Parts:
- added H1: MountingHole_2.2mm_M2, MountingHole_2.2mm_M2, F.Cu at (22.0, 25.7)
- added H2: MountingHole_2.2mm_M2, MountingHole_2.2mm_M2, F.Cu at (22.0, 38.2)
- added H3: MountingHole_2.2mm_M2, MountingHole_2.2mm_M2, F.Cu at (43.0, 25.7)
- added H4: MountingHole_2.2mm_M2, MountingHole_2.2mm_M2, F.Cu at (43.0, 38.2)
